File: PCB design for Quadrarure oscillator/Final PCB for 1khz Sine wave generator 2.kicad_pcb (KiCad board)
At the start: 2 copper layers, 36 x 60.5 mm, 20 parts, among them J1 Screw_Terminal_01x02, J2 Screw_Terminal_01x02, U1 LM358

Commit message: Add files via upload
Parts:
- moved G*** 0.71 mm to (167.0, 71.5)
Connections:
- RV1 pad 1: Net-(U1A--) -> unconnected-(RV1-Pad1)
- RV1 pad 2: unconnected-(RV1-Pad2) -> Net-(U1A--)
- RV2 pad 1: Sine Output -> unconnected-(RV2-Pad1)
- RV2 pad 2: unconnected-(RV2-Pad2) -> Sine Output
- RV3 pad 2: unconnected-(RV3-Pad2) -> Net-(U1B-+)
- RV3 pad 3: Net-(U1B-+) -> unconnected-(RV3-Pad3)
- RV4 pad 1: Net-(D1-K) -> unconnected-(RV4-Pad1)
- RV4 pad 2: unconnected-(RV4-Pad2) -> Net-(D1-K)
- RV7 pad 2: unconnected-(RV7-Pad2) -> Net-(D2-K)
- RV7 pad 3: Net-(D2-K) -> unconnected-(RV7-Pad3)
- RV7 pad 4: Net-(D1-A) -> unconnected-(RV7-Pad4)
- RV7 pad 5: unconnected-(RV7-Pad5) -> Net-(D1-A)
Routing:
- net Net-(U1B-+): track 23.7 -> 17.3 mm, vias 1 -> 0
- net Net-(D1-A): track 45.3 -> 40.2 mm, vias 1 -> 0
- net GNDREF: track 42.9 -> 38.8 mm
- net Sine Output: track 65.8 -> 61.9 mm, vias 0 -> 1
- net Net-(D1-K): track 45.7 -> 49.2 mm
- net Vin+: track 78.6 -> 80.6 mm, vias 0 -> 1
- net Net-(U1A--): track 29.5 -> 30.6 mm
- net Cosine Output: track 54.2 -> 53.5 mm
Other:
- board size 36 x 60.5 mm -> 36 x 61.5 mm
