File: PCB design for Quadrarure oscillator/Final PCB for 1khz Sine wave generator 2.kicad_sch (KiCad schematic)
At the start: 19 parts, among them J1 Screw_Terminal_01x02, J2 Screw_Terminal_01x02, U1 LM358

Commit message: Add files via upload
Parts:
- RV7: footprint Potentiometer_THT:Potentiometer_Vishay_148-149_Dual_Horizontal -> Potentiometer_THT:Potentiometer_Alps_RK163_Dual_Horizontal
Connections:
- net Sine Output: now also RV2.2; no longer RV2.1
- net at D2.1 (K), R3.1: now also RV7.2; no longer RV7.3
- net at C5.2, D1.1 (K), D2.2 (A)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: now also RV4.2; no longer RV4.1
- net at C3.2, U1.2 (-): now also RV1.2; no longer RV1.1
- net at D1.2 (A), R4.2: now also RV7.5; no longer RV7.4
- net at U1.5 (+): now also RV3.2; no longer RV3.3
